Commit message: update cart

File: example/urdf/ign_robot.urdf (robot description, URDF)
Before this commit: robot diff_drive, 11 links, 10 joints
Links:
- removed link cart_real
- added link cart_board, mass 1; collision box size=1.0 1.0 0.01; visual box size=1.0 1.0 0.01
- added link cart_hinge, mass 1; collision box size=0.1 0.1 0.01; visual box size=0.1 0.1 0.01
- added link cart_left, mass 1; collision box size=0.5 1.0 0.01; visual box size=0.5 1.0 0.01
- added link cart_right, mass 1; collision box size=0.5 1.0 0.01; visual box size=0.5 1.0 0.01
Joints:
- removed joint cart_to_cart_real
- added joint cart_joint_left: type fixed, parent cart_board, child cart_left, origin xyz=0 0.5 0.25 rpy=0 1.57 1.57
- added joint cart_joint_right: type fixed, parent cart_board, child cart_right, origin xyz=0 -0.5 0.25 rpy=0 1.57 1.57
- added joint cart_to_cart_hinge: type revolute, parent cart, child cart_hinge, origin xyz=-0.1 0 0 rpy=0 0 -1.57, limit lower=0.0 upper=0.548 effort=1000.0 velocity=0.5
- added joint cartreal_to_board: type fixed, parent cart_hinge, child cart_board, origin xyz=0 -0.5 0 rpy=0 0 1.57
- joint chassis_to_leg1: origin xyz=-1.5 0.0 0.2 rpy=0 0.5 0 -> xyz=-1.55 0.0 0.14 rpy=0 0.5 0

Commit message: add camera

File: example/urdf/ign_robot.urdf (robot description, URDF)
Before this commit: robot diff_drive, 14 links, 13 joints
Links:
- added link front_camera; visual box size=0.1 0.1 0.1
Joints:
- added joint front_camera_joint: type fixed, parent chassis, child front_camera, origin xyz=1.2 0 0.82 rpy=0 0 0
